Commit message: order in default.xacro

File: my_robot/urdf/default.xacro (robot description, xacro)
@@ -1,16 +1,4 @@
 <?xml version='1.0'?>
 <robot name="my_robot" xmlns:xacro="http://www.ros.org/wiki/xacro">
-<!--
-	<xacro:property name="base_link_x" value="0.44"/>
-	<xacro:property name="base_link_y" value="0.3"/>
-	<xacro:property name="base_link_z" value="0.076"/>
-	<xacro:property name="base_link_mass" value="10.0"/>
-	<xacro:property name="base_origin_xyz" value="0 0 0"/>
-	<xacro:property name="base_origin_rpy" value="0.0 0 0.0"/>
-	<xacro:property name="base_link_name" value="base_link"/>
-	<xacro:property name="base_link_wheel_offset_x" value="0.0"/>
-	<xacro:property name="base_link_wheel_offset_y" value="0.05"/>
-	<xacro:property name="base_link_wheel_offset_z" value="0.00"/>
-	-->
 	<xacro:property name="wheel_radius" value="0.1"/>
 	<xacro:property name="wheel_heigth" value="0.05"/>
@@ -18,26 +6,3 @@
 	<xacro:property name="wheel_origin_angle" value="0 1.5707 1.5707"/>
 	<xacro:property name="wheel_origin_position" value="0 0 0"/>
-<!--
-	<xacro:property name="mecanum_wheel_radius" value="0.01"/>
-	<xacro:property name="mecanum_wheel_mass" value="0.5"/>
-	<xacro:property name="mecanum_wheel_origin_angle_r" value="0"/>
-	<xacro:property name="mecanum_wheel_origin_angle_p" value="1.5707"/>
-	<xacro:property name="mecanum_wheel_origin_angle_y" value="0.785398"/>
-	<xacro:property name="mecanum_wheel_origin_position" value="0 0 0"/>
-	<xacro:property name="arm_size_x" value="0.2"/>
-	<xacro:property name="arm_size_y" value="0.1"/>
-	<xacro:property name="arm_size_z" value="0.05"/>
-	<xacro:property name="arm_wheel_offset_x" value="0.0"/>
-	<xacro:property name="arm_wheel_offset_y" value="0.0"/>
-	<xacro:property name="arm_wheel_offset_z" value="0.0"/>
-	<xacro:property name="wheel_mechanical_reduction" value="1"/>
-	<xacro:property name="arm_mecanum_wheel_offset_x" value="0.0"/>
-	<xacro:property name="arm_mecanum_wheel_offset_y" value="-0.1"/>
-	<xacro:property name="arm_mecanum_wheel_offset_z" value="0.05"/>
-	<xacro:property name="arm_joint_offset_x" value="-0.02"/>
-	<xacro:property name="arm_joint_offset_y" value="0.05"/>
-	<xacro:property name="kinect_joint_offset_x" value="${base_link_x/2+arm_size_x}"/>
-	<xacro:property name="kinect_joint_offset_y" value="0"/>
-	<xacro:property name="kinect_joint_offset_z" value="${arm_size_x}"/>
--->
 </robot>
