Commit message: changes in order in model

File: my_robot/urdf/my_robot.xacro (robot description, xacro)
@@ -10,7 +10,7 @@
 <xacro:include filename="lidar.xacro" />
 <!--<xacro:wheel side="left" />-->
-	<xacro:wheel_with_joint parent_name="chassis" pre_name="base" frontal_name="link" left="1" radius="${wheel_radius}" heigth="${wheel_heigth}" jointX="0" jointY="0.15" jointZ="0">
+	<xacro:wheel_with_joint parent_name="chassis" left="1" radius="${wheel_radius}" heigth="${wheel_heigth}" jointX="0" jointY="0.15" jointZ="0">
 	</xacro:wheel_with_joint>
-    <xacro:wheel_with_joint parent_name="chassis" pre_name="base" frontal_name="link" left="0" radius="${wheel_radius}" heigth="${wheel_heigth}" jointX="0" jointY="0.15" jointZ="0">
+    <xacro:wheel_with_joint parent_name="chassis" left="0" radius="${wheel_radius}" heigth="${wheel_heigth}" jointX="0" jointY="0.15" jointZ="0">
 	</xacro:wheel_with_joint>
     <xacro:camera name="camera" />

File: my_robot/urdf/wheel_with_joint.xacro (robot description, xacro)
@@ -1,5 +1,5 @@
 <?xml version='1.0'?>
 <robot name="my_robot" xmlns:xacro="http://www.ros.org/wiki/xacro">
-	<xacro:macro name="wheel_with_joint" params="parent_name frontal_name pre_name left radius heigth jointX jointY jointZ">
+	<xacro:macro name="wheel_with_joint" params="parent_name left radius heigth jointX jointY jointZ">
 		<xacro:property name="name_side" value="right"/>
 		<xacro:property name="reflect_side" value="-1"/>
