Commit message: Changes in model

File: my_robot/urdf/chasis.xacro (robot description, xacro)
@@ -21,5 +21,6 @@
       <origin xyz="0 0 0" rpy=" 0 0 0"/>
       <geometry>
-        <box size=".4 .2 .1"/>
+        <!--<box size="${chassis_box_x} ${chassis_box_y} ${chassis_box_z}"/>-->
+        <cylinder radius="${chassis_r}" length="${chassis_h}"/>
       </geometry>
     </collision>
@@ -27,29 +28,30 @@
       <origin xyz="0 0 0" rpy=" 0 0 0"/>
       <geometry>
-        <box size=".4 .2 .1"/>
+        <!--<box size="${chassis_box_x} ${chassis_box_y} ${chassis_box_z}"/>-->
+        <cylinder radius="${chassis_r}" length="${chassis_h}"/>
       </geometry>
     </visual>
     <collision name='back_caster_collision'>
-      <origin xyz="-0.15 0 -0.05" rpy=" 0 0 0"/>
+      <origin xyz="${-chassis_r+0.05} 0 ${-chassis_h/2}" rpy=" 0 0 0"/>
       <geometry>
-        <sphere radius="0.0499"/>
+        <sphere radius="${wheel_radius-chassis_h/2}"/>
       </geometry>
     </collision>
     <visual name='back_caster_visual'>
-      <origin xyz="-0.15 0 -0.05" rpy=" 0 0 0"/>
+      <origin xyz="${-chassis_r+0.05} 0 ${-chassis_h/2}" rpy=" 0 0 0"/>
       <geometry>
-        <sphere radius="0.05"/>
+        <sphere radius="${wheel_radius-chassis_h/2}"/>
       </geometry>
     </visual>
     <collision name='front_caster_collision'>
-      <origin xyz="0.15 0 -0.05" rpy=" 0 0 0"/>
+      <origin xyz="${+chassis_r-0.05} 0 ${-chassis_h/2}" rpy=" 0 0 0"/>
       <geometry>
-        <sphere radius="0.0499"/>
+        <sphere radius="${wheel_radius-chassis_h/2}"/>
       </geometry>
     </collision>
     <visual name='front_caster_visual'>
-      <origin xyz="0.15 0 -0.05" rpy=" 0 0 0"/>
+      <origin xyz="${+chassis_r-0.05} 0 ${-chassis_h/2}" rpy=" 0 0 0"/>
       <geometry>
-        <sphere radius="0.05"/>
+        <sphere radius="${wheel_radius-chassis_h/2}"/>
       </geometry>
     </visual>

File: my_robot/urdf/default.xacro (robot description, xacro)
@@ -1,8 +1,10 @@
 <?xml version='1.0'?>
 <robot name="my_robot" xmlns:xacro="http://www.ros.org/wiki/xacro">
-	<xacro:property name="wheel_radius" value="0.1"/>
+	<xacro:property name="wheel_radius" value="0.07"/>
 	<xacro:property name="wheel_heigth" value="0.05"/>
 	<xacro:property name="wheel_mass" value="5"/>
 	<xacro:property name="wheel_origin_angle" value="0 1.5707 1.5707"/>
 	<xacro:property name="wheel_origin_position" value="0 0 0"/>
+	<xacro:property name="chassis_r" value=".2"/>
+	<xacro:property name="chassis_h" value=".1"/>
 </robot>

File: my_robot/urdf/my_robot.xacro (robot description, xacro)
@@ -10,7 +10,7 @@
 <xacro:include filename="lidar.xacro" />
 <!--<xacro:wheel side="left" />-->
-	<xacro:wheel_with_joint parent_name="chassis" left="1" radius="${wheel_radius}" heigth="${wheel_heigth}" jointX="0" jointY="0.15" jointZ="0">
+	<xacro:wheel_with_joint parent_name="chassis" left="1" radius="${wheel_radius}" heigth="${wheel_heigth}" jointX="0" jointY="${chassis_r+wheel_heigth}" jointZ="0">
 	</xacro:wheel_with_joint>
-    <xacro:wheel_with_joint parent_name="chassis" left="0" radius="${wheel_radius}" heigth="${wheel_heigth}" jointX="0" jointY="0.15" jointZ="0">
+    <xacro:wheel_with_joint parent_name="chassis" left="0" radius="${wheel_radius}" heigth="${wheel_heigth}" jointX="0" jointY="${chassis_r+wheel_heigth}" jointZ="0">
 	</xacro:wheel_with_joint>
     <xacro:camera name="camera" />
